File: kicad/octaver/octaver.sch (KiCad schematic (older format))
At the start: 70 parts, among them IC1 X9C104SIZ, IC2 ISL21080CIH315Z-TK, J1 NMJ4HCD2, J2 NMJ4HCD2, J3 audio input, J4 POT_CON, J5 Power In, U1 NE5532, U2 NE5532, U3 NE5532, U4 NE5532, U5 NE5532, U6 AMS1117-5.0, U7 AMS1117-3.3, U8 NUCLEO64-F411RE

Commit message: Added resque files
Parts:
- IC1: symbol downloaded:X9C104SIZ -> octaver-rescue:X9C104SIZ-downloaded
- IC2: symbol downloaded:ISL21080CIH315Z-TK -> octaver-rescue:ISL21080CIH315Z-TK-downloaded
- J1, J2: symbol downloaded:NMJ4HCD2 -> octaver-rescue:NMJ4HCD2-downloaded
Changed lines of the file:
@@
 $EndComp
 $Comp
-L downloaded:X9C104SIZ IC1
+L octaver-rescue:X9C104SIZ-downloaded IC1
 U 1 1 618490AD
 P 800 4650
@@
 	5400 3450 5350 3450
 $Comp
-L downloaded:NMJ4HCD2 J1
+L octaver-rescue:NMJ4HCD2-downloaded J1
 U 1 1 6187ED00
 P 1200 1950
@@
 Connection ~ 4850 3200
 $Comp
-L downloaded:NMJ4HCD2 J2
+L octaver-rescue:NMJ4HCD2-downloaded J2
 U 1 1 61E3A7DE
 P 2200 7350
@@
 Connection ~ 6900 4300
 $Comp
-L downloaded:ISL21080CIH315Z-TK IC2
+L octaver-rescue:ISL21080CIH315Z-TK-downloaded IC2
 U 1 1 623CF186
 P 6650 5750
